File: dcload-interface-board/schematics/display.kicad_sch (KiCad schematic)
At the start: 13 parts, among them U300 WEO012864L

Commit message: add: interface panel board
Other:
- title: Linear PSU Digital Board -> Display
